File: Circuit-Diagram/Articulated-Robot/Articulated-Robot.kicad_sch (KiCad schematic)
At the start: 0 parts

Commit message: Made and ordered a pcb for the circuit.
Parts:
- added A1: Arduino_Nano_v3.x, Module:Arduino_Nano_WithMountingHoles, symbol MCU_Module:Arduino_Nano_v3.x
- added C1: 470µ, Capacitor_THT:CP_Radial_D6.3mm_P2.50mm, symbol Device:C_Polarized
- added C2, C3, C4, C5: 100n, Capacitor_THT:C_Disc_D4.3mm_W1.9mm_P5.00mm, symbol Device:C
- added J1: Base Motor, Connector_PinHeader_2.54mm:PinHeader_1x03_P2.54mm_Vertical, symbol Connector_Generic:Conn_01x03
- added J2: Shoulder Motor, Connector_PinHeader_2.54mm:PinHeader_1x03_P2.54mm_Vertical, symbol Connector_Generic:Conn_01x03
- added J3: Elbow Motor, Connector_PinHeader_2.54mm:PinHeader_1x03_P2.54mm_Vertical, symbol Connector_Generic:Conn_01x03
- added J4: Barrel_Jack_5.5x2.1mm, Connector_BarrelJack_2:Barrel_Jack_5.5x2.1mm, symbol Connector_BarrelJack_2:Barrel_Jack
- added SW1: SW_Push_Dual, Button_Switch_THT:SW_PUSH_6mm_H4.3mm, symbol Switch:SW_Push_Dual
Connections:
- new net: A1.5 (D2), C2.2, SW1.2
- new net: A1.6 (D3), J1.1 (Pin_1)
- new net: A1.9 (D6), J3.1 (Pin_1)
- new net: A1.8 (D5), J2.1 (Pin_1)
- new net +5V: A1.27 (+5V)
- new net GND: A1.29 (GND), A1.4 (GND), C1.2, C2.1, C3.1, C4.1, C5.1, J1.3 (Pin_3), J2.3 (Pin_3), J3.3 (Pin_3), J4.2, SW1.1
- new net VCC: C1.1, C3.2, C4.2, C5.2, J1.2 (Pin_2), J2.2 (Pin_2), J3.2 (Pin_2), J4.1
- no-connect marks 0 -> 25
